File: velion_lightboard_pcb.kicad_sch (KiCad schematic)
At the start: 0 parts

Commit message: designing relay board
Parts:
- added C1, C2: 100nF, Capacitor_SMD:C_1206_3216Metric_Pad1.33x1.80mm_HandSolder, symbol Device:C
- added D4: US1M, Diode_SMD:D_SMA, symbol Diode:US1M
- added D5: WS2812B, LED_SMD:LED_WS2812B_PLCC4_5.0x5.0mm_P3.2mm, symbol LED:WS2812B
- added J1, J2: Conn_01x04, velion_mainboard:15EDG-4P, symbol Connector_Generic:Conn_01x04
- added J10, J11, J3, J4, J5, J6, J7, J8, J9: Conn_01x03, symbol Connector_Generic:Conn_01x03
- added Q1, Q2, Q3, Q4, Q5, Q6, Q7, Q8: NMOS, Package_TO_SOT_SMD:SOT-23, symbol Transistor_FET_Other:Q_NMOS_Depletion_GSD
- added R1, R10, R11, R12, R13, R2, R8, R9: 10K, symbol Device:R
- added R14, R15, R16, R17, R19, R20, R21, R22: 0.001 R, symbol Device:R
- added R18: 120 R, Resistor_SMD:R_1206_3216Metric_Pad1.30x1.75mm_HandSolder, symbol Device:R
- added R3, R4, R5: 100R, Resistor_SMD:R_1206_3216Metric_Pad1.30x1.75mm_HandSolder, symbol Device:R
- added R6, R7: 4k7, Resistor_SMD:R_1206_3216Metric_Pad1.30x1.75mm_HandSolder, symbol Device:R
- added U1: TJA1051T-3, Package_SO:SOIC-8_3.9x4.9mm_P1.27mm, symbol Interface_CAN_LIN:TJA1051T-3
- added U6: ESP32-DEVKITC-32D, velion_mainboard:MODULE_ESP32-DEVKITC-32D, symbol ESP32-DEVKITC-32D:ESP32-DEVKITC-32D
- added U7, U8: MCP23017_SO, Package_SO:SOIC-28W_7.5x17.9mm_P1.27mm, symbol Interface_Expansion:MCP23017_SO
Connections:
- new net: J8.2 (Pin_2), Q4.3 (D), R10.2
- new net: J5.2 (Pin_2), Q1.3 (D), R2.2
- new net: J11.2 (Pin_2), Q7.3 (D), R13.2
- new net: J9.2 (Pin_2), Q5.3 (D), R11.2
- new net: R5.2, U6.J3-14 (IO0)
- new net: J4.2 (Pin_2), Q8.3 (D), R1.2
- new net: J7.2 (Pin_2), Q3.3 (D), R9.2
- new net: J10.2 (Pin_2), Q6.3 (D), R12.2
- new net: R3.2, U6.J3-16 (IO15)
- new net: J6.2 (Pin_2), Q2.3 (D), R8.2
- new net: D4.1 (K), D5.1 (VDD)
- new net: R4.2, U6.J3-15 (IO2)
- new net: D5.2 (DOUT), J3.2 (Pin_2)
- new net +12V: J10.1 (Pin_1), J11.1 (Pin_1), J4.1 (Pin_1), J5.1 (Pin_1), J6.1 (Pin_1), J7.1 (Pin_1), J8.1 (Pin_1), J9.1 (Pin_1), R1.1, R10.1, R11.1, R12.1, R13.1, R2.1, R8.1, R9.1
- new net +3.3V: C1.1, R6.1, R7.1, U1.5 (VIO), U6.J2-1 (3V3), U7.15 (A0), U7.18 (~{RESET}), U7.9 (VDD), U8.18 (~{RESET}), U8.9 (VDD)
- new net +5V: C2.1, D4.2 (A), J3.1 (Pin_1), U1.3 (VCC), U6.J2-19 (EXT_5V)
- new net CANH: J1.3 (Pin_3), J2.3 (Pin_3), R18.1, U1.7 (CANH)
- new net CANL: J1.2 (Pin_2), J2.2 (Pin_2), R18.2, U1.6 (CANL)
- new net CAN_RX: U1.4 (RXD), U6.J3-8 (IO19)
- new net CAN_S: U1.8 (S), U6.J2-13 (IO12)
- new net CAN_TX: U1.1 (TXD), U6.J3-9 (IO18)
- new net GND: C1.2, C2.2, D5.3 (VSS), J1.1 (Pin_1), J2.1 (Pin_1), J3.3 (Pin_3), R14.2, R15.2, R16.2, R17.2, R19.2, R20.2, R21.2, R22.2, U1.2 (GND), U6.J2-14 (GND1), U6.J3-1 (GND3), U6.J3-7 (GND2), U7.10 (VSS), U7.16 (A1), U7.17 (A2), U8.10 (VSS), U8.15 (A0), U8.16 (A1), U8.17 (A2)
- new net LATCH_TRUNK_MOSFET_GATE: Q1.1 (G), Q2.1 (G), Q3.1 (G), Q4.1 (G), Q5.1 (G), Q6.1 (G), Q7.1 (G), Q8.1 (G)
- new net RGBLED_DIN: D5.4 (DIN), U6.J3-6 (IO21)
- new net SCL: R7.2, U6.J3-3 (IO22), U7.12 (SCK), U8.12 (SCK)
- new net SDA: R6.2, U6.J3-2 (IO23), U7.13 (SDA), U8.13 (SDA)
- new net SENSE: J10.3 (Pin_3), J11.3 (Pin_3), J4.3 (Pin_3), J5.3 (Pin_3), J6.3 (Pin_3), J7.3 (Pin_3), J8.3 (Pin_3), J9.3 (Pin_3), Q1.2 (S), Q2.2 (S), Q3.2 (S), Q4.2 (S), Q5.2 (S), Q6.2 (S), Q7.2 (S), Q8.2 (S), R14.1, R15.1, R16.1, R17.1, R19.1, R20.1, R21.1, R22.1
- new net VBUS: J1.4 (Pin_4), J2.4 (Pin_4)
- no-connect marks 0 -> 13
Other:
- note added: "0100000 = 0x20"
- note added: "0100001 = 0x21"
- note added: "3v3 provided by internal LDO of ESP32 devboard"
- note added: "5A MAX"
- note added: "CAN BUS Power Rail"
- note added: "CAN IN"
- note added: "CAN OUT"
- note added: "CAN Transceiver"
- note added: "Compute"
- note added: "Never powered Down so that emergency signal keep blinking"
- note added: "RGB strip"
- note added: "add ADC here with 8 channel"
- note added: "daylight sensor"
- note added: "diode -> little hack to drive the WS2812 using 3v3 logic"
- note added: "https://hackaday.com/2017/01/20/cheating-at-5v-ws2812-control-to-use-a-3-3v-data-line/"
- note added: "leave serial port for debug"
- note added: "proximity sensor"
- note added: "resistor to limit risk of issue due to current leakage and the mosfet grid capacitor that could influence the strapping pin at boot."
- note added: "size R for 20 mA or better of resolution keep power below 0.1 W -> max 20 mV max 0.004 mR"
- note added: "small sig 20 V 5A mosfet"
- note added: "switch to ESP32 C3 super micro"
